File: LPC55Sxx.sch (KiCad schematic (older format))
At the start: 17 parts, among them J1 DNP, J3 Conn_01x05, U1 LPC55S69JEV98K, U3 SE050, Y1 XRCGB16M000FXN01R0

Commit message: nk3cn423
Parts:
- removed J1: DNP, nitro:molex78646-3001, symbol Connector:SIM_Card
- added TP3, TP4: TestPoint, TestPoint:TestPoint_Pad_1.5x1.5mm, symbol Connector:TestPoint
- U1: symbol solo-A-rescue:LPC55S69JEV98K-solo-solo-A-rescue -> nk3cn-zeus-rescue:LPC55S69JEV98K-solo-solo-A-rescue-solo-A-rescue-fido2-lpc55-rescue; Manufacturer NXP USA Inc. -> NXP
- U3: symbol SE050:SE050 -> nk3cn-zeus-rescue:SE050-SE050; MPN SE050C1HQ1/Z01SCZ -> (none); Manufacturer NXP -> (none); Package 20-HX2QFN (3x3) -> (none); Pins 20 -> (none)
Connections:
- wire segments 131 -> 133
- no-connect marks 7 -> 6
Changed lines of the file:
@@
 $EndComp
 Wire Wire Line
-	9900 1300 9650 1300
+	9900 1300 9800 1300
 $Comp
 L power:GNDREF #PWR0104
@@
 G
 $Comp
-L solo-A-rescue:LPC55S69JEV98K-solo-solo-A-rescue U1
+L nk3cn-zeus-rescue:LPC55S69JEV98K-solo-solo-A-rescue-solo-A-rescue-fido2-lpc55-rescue U1
 U 1 1 5E727C5A
 P 2900 2500
@@
 F 1 "LPC55S69JEV98K" H 2493 726 50  0000 C CNN
 F 2 "solo:BGA98C50P13X13_700X700X97N" H 2900 2500 50  0001 L BNN
-F 3 "" H 2900 2500 50  0001 L BNN
+F 3 "NXP USA Inc." H 2900 2500 50  0001 L BNN
 F 4 "LPC55S69 ARM 32-bit M33 TrustZone" H 2900 2500 50  0001 L BNN "Description"
-F 5 "NXP USA Inc." H 2900 2500 50  0001 L BNN "Manufacturer"
+F 5 "NXP" H 2900 2500 50  0001 L BNN "Manufacturer"
 F 6 "LPC55S69JEV98K" H 2900 2500 50  0001 L BNN "MPN"
 F 7 "98" H 2900 2500 50  0001 L BNN "Pins"
@@
 $EndComp
 $Comp
-L solo-A-rescue:LPC55S69JEV98K-solo-solo-A-rescue U1
+L nk3cn-zeus-rescue:LPC55S69JEV98K-solo-solo-A-rescue-solo-A-rescue-fido2-lpc55-rescue U1
 U 2 1 5E72B48A
 P 2300 6100
@@
 F 1 "LPC55S69JEV98K" H 1653 4326 50  0000 C CNN
 F 2 "solo:BGA98C50P13X13_700X700X97N" H 2300 6100 50  0001 L BNN
-F 3 "" H 2300 6100 50  0001 L BNN
+F 3 "NXP USA Inc." H 2300 6100 50  0001 L BNN
 F 4 "LPC55S69 ARM 32-bit M33 TrustZone" H 2300 6100 50  0001 L BNN "Description"
-F 5 "NXP USA Inc." H 2300 6100 50  0001 L BNN "Manufacturer"
+F 5 "NXP" H 2300 6100 50  0001 L BNN "Manufacturer"
 F 6 "LPC55S69JEV98K" H 2300 6100 50  0001 L BNN "MPN"
 F 7 "98" H 2300 6100 50  0001 L BNN "Pins"
@@
 $EndComp
 $Comp
-L solo-A-rescue:LPC55S69JEV98K-solo-solo-A-rescue U1
+L nk3cn-zeus-rescue:LPC55S69JEV98K-solo-solo-A-rescue-solo-A-rescue-fido2-lpc55-rescue U1
 U 3 1 5E72DEEE
 P 8600 5000
@@
 F 1 "LPC55S69JEV98K" H 8550 6176 50  0000 C CNN
 F 2 "solo:BGA98C50P13X13_700X700X97N" H 8600 5000 50  0001 L BNN
-F 3 "" H 8600 5000 50  0001 L BNN
+F 3 "NXP USA Inc." H 8600 5000 50  0001 L BNN
 F 4 "LPC55S69 ARM 32-bit M33 TrustZone" H 8600 5000 50  0001 L BNN "Description"
-F 5 "NXP USA Inc." H 8600 5000 50  0001 L BNN "Manufacturer"
+F 5 "NXP" H 8600 5000 50  0001 L BNN "Manufacturer"
 F 6 "LPC55S69JEV98K" H 8600 5000 50  0001 L BNN "MPN"
 F 7 "98" H 8600 5000 50  0001 L BNN "Pins"
@@
 	7600 5900 7600 6150
 NoConn ~ 7700 6000
-$Comp
-L Connector:SIM_Card J1
-U 1 1 5F2172A8
-P 8050 3350
-F 0 "J1" H 8680 3450 50  0000 L CNN
-F 1 "DNP" H 8680 3359 50  0000 L CNN
-F 2 "nitro:molex78646-3001" H 8050 3700 50  0001 C CNN
-F 3 " ~" H 8000 3350 50  0001 C CNN
-	1    8050 3350
-	1    0    0    -1
-$EndComp
-$Comp
-L power:GNDREF #PWR0130
-U 1 1 5F2E34C8
-P 7550 3350
-F 0 "#PWR0130" H 7550 3100 50  0001 C CNN
-F 1 "GNDREF" V 7555 3222 50  0000 R CNN
-F 2 "" H 7550 3350 50  0001 C CNN
-F 3 "" H 7550 3350 50  0001 C CNN
-	1    7550 3350
-	0    1    1    0
-$EndComp
 Wire Wire Line
 	6200 2500 6450 2500
 Text Label 6450 2500 0    50   ~ 0
 SIM_CLK
-Text Label 7550 3250 2    50   ~ 0
-SIM_CLK
 Wire Wire Line
 	6200 2400 6450 2400
 Text Label 6450 2400 0    50   ~ 0
 SIM_IO
-Text Label 7550 3550 2    50   ~ 0
-SIM_IO
 Wire Wire Line
 	5000 6200 5100 6200
 Text Label 5100 6200 0    50   ~ 0
 SIM_RST
-Text Label 7550 3150 2    50   ~ 0
-SIM_RST
-NoConn ~ 7550 3450
-Text Label 7550 3050 2    50   ~ 0
-SIM_VCC
 Text Label 6500 3200 0    50   ~ 0
 SIM_VCC
@@
 $EndComp
 $Comp
-L SE050:SE050 U3
+L nk3cn-zeus-rescue:SE050-SE050 U3
 U 1 1 5F974D56
 P 8050 2300
+AR Path="/5F974D56" Ref="U3"  Part="1"
+AR Path="/5DDFB633/5DDC9C59/5F974D56" Ref="U3"  Part="1"
 F 0 "U3" H 8150 1811 50  0000 C CNN
 F 1 "SE050" H 8150 1720 50  0000 C CNN
 F 2 "Package_DFN_QFN:UQFN-20-1EP_3x3mm_P0.4mm_EP1.85x1.85mm" H 8050 2300 50  0001 C CNN
 F 3 "" H 8050 2300 50  0001 C CNN
-F 4 "SE050C1HQ1/Z01SCZ" H 8050 2300 50  0001 C CNN "MPN"
-F 5 "NXP" H 8050 2300 50  0001 C CNN "Manufacturer"
-F 6 "20-HX2QFN (3x3)" H 8050 2300 50  0001 C CNN "Package"
-F 7 "20" H 8050 2300 50  0001 C CNN "Pins"
 	1    8050 2300
 	1    0    0    -1
@@
 Wire Wire Line
 	6400 3600 6200 3600
+$Comp
+L Connector:TestPoint TP3
+U 1 1 5FB61888
+P 9750 1300
+F 0 "TP3" V 9945 1372 50  0000 C CNN
+F 1 "TestPoint" V 9854 1372 50  0000 C CNN
+F 2 "TestPoint:TestPoint_Pad_1.5x1.5mm" H 9950 1300 50  0001 C CNN
+F 3 "~" H 9950 1300 50  0001 C CNN
+	1    9750 1300
+	-1   0    0    1
+$EndComp
+Connection ~ 9750 1300
+Wire Wire Line
+	9750 1300 9650 1300
+$Comp
+L Connector:TestPoint TP4
+U 1 1 5FB76D8F
+P 9800 1300
+F 0 "TP4" V 9995 1372 50  0000 C CNN
+F 1 "TestPoint" V 9904 1372 50  0000 C CNN
+F 2 "TestPoint:TestPoint_Pad_1.5x1.5mm" H 10000 1300 50  0001 C CNN
+F 3 "~" H 10000 1300 50  0001 C CNN
+	1    9800 1300
+	-1   0    0    1
+$EndComp
+Connection ~ 9800 1300
+Wire Wire Line
+	9800 1300 9750 1300
 $EndSCHEMATC
