File: solo.sch (KiCad schematic (older format))
At the start: 18 parts, among them J2 Conn_01x04, T1 TLV742p, U2 MTCH101

Commit message: nk3cn423
Parts:
- removed CX2: 36pF, Capacitor_SMD:C_0402_1005Metric, symbol Device:C
- removed R5, R7: 4.7k, Resistor_SMD:R_0402_1005Metric, symbol Device:R
- removed R8: DNP, Resistor_SMD:R_0402_1005Metric, symbol Device:R
- removed U2: MTCH101, Package_TO_SOT_SMD:SOT-23-6, symbol solo-A-rescue:MTCH101-nk-fido2
- added C5: 20pF, Capacitor_SMD:C_0402_1005Metric, symbol Device:C
- added CY1: DNP, Capacitor_SMD:C_0402_1005Metric, symbol Device:C
- added U2: TTP233D-HA6, Package_TO_SOT_SMD:TSOT-23-6, symbol corelib:TTP233
- C1, C3, C4: value 10u -> 22u
- C2: value 100n -> 100nF
- CX1: Description 100pF 5% -> (none)
- F1: symbol solo-A-rescue:quad_serial_flash-solo-solo-A-rescue -> nk3cn-zeus-rescue:quad_serial_flash-solo-solo-A-rescue-solo-A-rescue-fido2-lpc55-rescue
- N1: footprint solo:MLPD3X3 -> Package_DFN_QFN:DFN-10-1EP_3x3mm_P0.5mm_EP1.55x2.48mm; symbol solo-A-rescue:FM11NC08-solo-solo-A-rescue -> nk3cn-zeus-rescue:FM11NC08-solo-solo-A-rescue-solo-A-rescue-fido2-lpc55-rescue
- R2: value 4.7k -> 1k
- T1: value TLV742p -> AP7340-33FS4-7; footprint solo:Texas_X2SON-4_1x1mm_P0.65mm -> corelib:Diodes_X2-DFN1010_1x1mm_P0.65mm; symbol solo-A-rescue:TLV742p-solo-solo-A-rescue -> nk3cn-zeus-rescue:TLV742p-solo-solo-A-rescue-solo-A-rescue-fido2-lpc55-rescue; MPN TLV74233PDQNR -> AP7340-33FS4-7; Manufacturer Texas Instruments -> Diodes, Inc; Package X2SON-4 -> AP7340-33FS4-7
Connections:
- wire segments 140 -> 133
- no-connect marks 3 -> 4
Other:
- moved on the sheet: R2
